File: PBJ_EU.kicad_pcb (KiCad board)
At the start: 2 copper layers, 111.4 x 128.5 mm, 39 parts, among them J1 Conn_02x06_Odd_Even, J6 Conn_02x08_Odd_Even_Female, SW3 Power

Commit message: v 10.4
Parts:
- J6: footprint Connector_PinHeader_2.54mm:PinHeader_2x08_P2.54mm_Vertical -> Connector_PinSocket_2.54mm:PinSocket_2x08_P2.54mm_Vertical
- moved J6 2.54 mm to (86.8, 123.0)
Connections:
- J6 pad 10: Tip3 -> SW3
- J6 pad 11: SW4 -> Tip4
- J6 pad 12: Tip4 -> SW4
- J6 pad 13: B Rail -> A Rail
- J6 pad 14: A Rail -> B Rail
- J6 pad 5: SW1 -> Tip1
- J6 pad 6: Tip1 -> SW1
- J6 pad 7: SW2 -> Tip2
- J6 pad 8: Tip2 -> SW2
- J6 pad 9: SW3 -> Tip3
Other:
- board text added: "S/N 10.4"
- board text added: "v10.4"
- board text removed: "OFF"
- board text removed: "S/N 10.3"
- board text removed: "v10.3"
