File: sub/sub.kicad_pcb (KiCad board)
At the start: 2 copper layers, 111.4 x 29.4 mm, 70 parts, among them J1 Thonk 3.5mm Jack, J2 Thonk 3.5mm Jack, J3 Thonk 3.5mm Jack, J4 Thonk 3.5mm Jack, J5 Conn_02x06_Odd_Even, J6 Conn_02x05_Odd_Even, Q1 PMV65XP, Q2 PMV65XP, Q3 AO3400A, Q4 AO3400A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

Commit message: v3.2
Parts:
- removed Q1, Q2: PMV65XP, Package_TO_SOT_SMD:SOT-23
- removed Q3, Q4: AO3400A, Package_TO_SOT_SMD:SOT-23
- removed R19, R20, R21, R22, R23, R24, R25, R26: 10K, Resistor_SMD:R_0402_1005Metric
- moved J6 11.4 mm to (92.4, 126.5)
Connections:
- SW4 pad 2: Net-(Q1-D) -> -12V
- SW4 pad 5: Net-(Q2-D) -> +12V
Routing:
- net Net-(Q2-D): track 33.7 -> 0.00 mm, vias 3 -> 0
- net Net-(Q1-D): track 27.7 -> 0.00 mm, vias 1 -> 0
- net +12V: track 125.9 -> 140.4 mm, vias 8 -> 4
- net Net-(J6-Pin_1): track 40.1 -> 28.7 mm
- net Net-(J6-Pin_10): track 29.6 -> 18.2 mm
- net Net-(Q2-G): track 5.58 -> 0.00 mm
- net -12V: track 113.4 -> 118.1 mm, vias 6 -> 4
- net Net-(Q4-G): track 4.43 -> 0.00 mm, vias 2 -> 0
- net GND: track 42.7 -> 39.9 mm, vias 27 -> 25
- net Net-(Q3-G): track 2.57 -> 0.00 mm
- net Net-(Q1-G): track 2.57 -> 0.00 mm
Other:
- board text added: "3.2."
- board text removed: "3.1."
- board text removed: "Either Way"

Commit message: v 10.4
Parts:
- added C15: 22uF, Capacitor_SMD:C_0805_2012Metric_Pad1.18x1.45mm_HandSolder, B.Cu at (89.2, 135.2)
- added C16: 22uF, Capacitor_SMD:C_0805_2012Metric_Pad1.18x1.45mm_HandSolder, B.Cu at (103.2, 126.8)
- added D2: 1N5819WS, Diode_SMD:D_SOD-323, B.Cu at (64.8, 129.5)
- added D4: 1N5819WS, Diode_SMD:D_SOD-323, B.Cu at (64.8, 122.5)
Connections:
- SW4 pad 2: -12V -> Net-(D4-K)
- SW4 pad 5: +12V -> Net-(D2-A)
Routing:
- net GND: track 39.9 -> 44.5 mm, vias 25 -> 26
- net Net-(D2-A): track 0.00 -> 2.22 mm
- net Net-(D4-K): track 0.00 -> 2.20 mm
- net +12V: track 140.4 -> 139.0 mm
- net -12V: track 118.1 -> 119.4 mm, vias 4 -> 5
