File: sub/sub.kicad_sch (KiCad schematic)
At the start: 74 parts, among them J1 Thonk 3.5mm Jack, J2 Thonk 3.5mm Jack, J3 Thonk 3.5mm Jack, J4 Thonk 3.5mm Jack, J5 Conn_02x06_Odd_Even, J6 Conn_02x05_Odd_Even, Q1 PMV65XP, Q2 PMV65XP, Q3 AO3400A, Q4 AO3400A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

Commit message: v3.2
Parts:
- removed Q1, Q2: PMV65XP, Package_TO_SOT_SMD:SOT-23, symbol Transistor_FET:BSS83P
- removed Q3, Q4: AO3400A, Package_TO_SOT_SMD:SOT-23, symbol Transistor_FET:AO3400A
- removed R19, R20, R21, R22, R23, R24, R25, R26: 10K, Resistor_SMD:R_0402_1005Metric, symbol Device:R_Small_US
- added SO5, SO6, SO7, SO8: LED Spacer, symbol Mechanical:MountingHole
- J6: Digi-Key Part S2011EC-05-ND -> S9169-ND
- R10, R14, R16, R8: Digi-Key Part CF14JT5K60CT-ND -> 541-2803-1-ND
- R11, R12, R17, R18: Digi-Key Part CF14JT1M00CT-ND -> 541-2803-1-ND
- R13, R15, R7, R9: Digi-Key Part RNCP0805FTD1K00CT-ND -> P17401CT-ND
- R3, R4: Digi-Key Part CF14JT20K0CT-ND -> 541-10449-1-ND
- U1, U3: Digi-Key Part 497-19621-ND -> 4518-LM317DCYRCT-ND
- U2, U4: Digi-Key Part 296-1775-5-ND -> 296-1282-1-ND
Connections:
- net +12V: now also SW4.5 (B)
- net -12V: now also SW4.2 (B)
Other:
- note added: "Note: Signal indicator LEDs (D1, D3 D5, D7) are installed so that Red indicates positive voltage and Green indicates negative. Switch the polarity of these LEDs to reverse the indication."
- note added: "note: the currently specd' blue LED doesn't fit in the spacer. The spacer is included in case a blue LED is found that fits."
- moved on the sheet: J5

Commit message: v 10.4
Parts:
- added C15, C16: 22uF, Capacitor_SMD:C_0805_2012Metric_Pad1.18x1.45mm_HandSolder, symbol Device:C_Small
- added D2, D4: 1N5819WS, Diode_SMD:D_SOD-323, symbol Diode:1N5819WS
Connections:
- net +12V: now also C16.2, D2.1 (K); no longer SW4.5 (B)
- net -12V: now also C15.1, D4.2 (A); no longer SW4.2 (B)
- net GND: now also C15.2, C16.1
- new net: D4.1 (K), SW4.2 (B)
- new net: D2.2 (A), SW4.5 (B)
Other:
- note added: "Caution! Shorting diodes removes reverse polarity protection."
- note added: "Input range: -12V ~ +12V"
- note added: "Short across diodes to get full voltage. Locations are marked by arrows on board."
- note removed: "Operating input range: -10V - +10V"
- title: (none) -> PBJ-EU
- moved on the sheet: J5, SW4A, SW4B

Commit message: Adds Sidecar v0.1
Parts:
- C15, C16, C3, C8: LCSC Part # C76637 -> C45783
- D2, D4: footprint Diode_SMD:D_SOD-323 -> Diode_SMD:D_SOD-123; LCSC Part # (none) -> C191023
Changed lines of the file:
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@@
 			)
 		)
-		(property "LCSC Part #" "C76637"
+		(property "LCSC Part #" "C45783"
 			(at 193.04 142.24 0)
 			(effects
@@
 			)
 		)
-		(property "LCSC Part #" "C76637"
+		(property "LCSC Part #" "C45783"
 			(at 113.03 151.13 0)
 			(effects
@@
 			)
 		)
-		(property "LCSC Part #" "C76637"
+		(property "LCSC Part #" "C45783"
 			(at 113.03 140.97 0)
 			(effects
@@
 			)
 		)
-		(property "Footprint" "Diode_SMD:D_SOD-323"
+		(property "Footprint" "Diode_SMD:D_SOD-123"
 			(at 85.09 161.925 0)
 			(effects
@@
 			)
 		)
+		(property "LCSC Part #" "C191023"
+			(at 85.09 157.48 0)
+			(effects
+				(font
+					(size 1.27 1.27)
+				)
+				(hide yes)
+			)
+		)
 		(pin "1"
 		)
@@
 			)
 		)
-		(property "Footprint" "Diode_SMD:D_SOD-323"
+		(property "Footprint" "Diode_SMD:D_SOD-123"
 			(at 85.09 130.175 0)
 			(effects
@@
 			)
 		)
+		(property "LCSC Part #" "C191023"
+			(at 85.09 134.62 0)
+			(effects
+				(font
+					(size 1.27 1.27)
+				)
+				(hide yes)
+			)
+		)
 		(pin "1"
 		)
@@
 			)
 		)
-		(property "LCSC Part #" "C76637"
+		(property "LCSC Part #" "C45783"
 			(at 254 142.24 0)
 			(effects
